File: Hardware/BirdAttractor_RevB/BirdAttractor_RevB.kicad_pcb (KiCad board)
At the start: 2 copper layers, 41 parts, among them P1 FTDI, P2 USB_B, P3 USB_A, P4 USB_A, Q1 BSS138, Q2 BSS138, SW1 SW_PUSH, SW2 SW_PUSH, U1 PR_Relay_V23079, U2 AMS1117-3.3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

Commit message: added pull down resistor to gpio15 for programming; created RevC and board ready for fabrication
Parts:
- added R21: 10K, Capacitors_SMD:C_1206, F.Cu at (158.0, 124.5)
- added R22: 10K, Capacitors_SMD:C_1206, F.Cu at (157.5, 114.0)
- BT1: footprint MyKiCadParts:BU2032-1-HD-G -> MyKiCadParts:BK-913
- R5: footprint LEDs:LED-3MM -> LEDs:LED-5MM
- moved BT1 11.8 mm to (196.0, 56.0)
Connections:
- U4 pad 11: (no net) -> RELAY_ON33
- U4 pad 12: (no net) -> RELAY_OFF33
- U4 pad 16: RELAY_ON33 -> Net-(R22-Pad1)
- U4 pad 17: RELAY_OFF33 -> Net-(R21-Pad1)
Routing:
- net RELAY_ON33: track 23.1 -> 3.21 mm
- net GND: track 51.4 -> 68.2 mm
- net VBAT: track 30.4 -> 13.5 mm
- net RELAY_OFF33: track 15.1 -> 6.54 mm
