File: Hardware/BirdAttractor_RevC/BirdAttractor_RevC.sch (KiCad schematic (older format))
At the start: 43 parts, among them P1 FTDI, P2 USB_B, P3 USB_A, P4 USB_A, Q1 BSS138, Q2 BSS138, SW1 SW_PUSH, SW2 SW_PUSH, U1 PR_Relay_V23079, U2 AMS1117-3.3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

Commit message: added pull down resistor to gpio15 for programming; created RevC and board ready for fabrication
Parts:
- removed R20: 0, Resistors_SMD:R_1206, symbol R
- removed U3: SN74LVC1G14, MyKiCadParts:SOT-23-5-80, symbol SN74LVC1G14
- removed U5: PCF2129AT, MyKiCadParts:SOIC-20_7.5x12.8mm_Pitch1.27mm-80, symbol PCF2129AT
- C1: value 1uF -> 10uF
- R9: value 100K -> 10K
- SW1: footprint Buttons_Switches_SMD:SW_SPST_PTS645 -> Buttons_Switches_ThroughHole:SW_PUSH_SMALL
Connections:
- wire segments 80 -> 77
Changed lines of the file:
@@
 LIBS:valves
 LIBS:myParts
-LIBS:BirdAttractor_RevB-cache
+LIBS:BirdAttractor_RevC-cache
 EELAYER 25 0
 EELAYER END
@@
 Sheet 1 1
 Title "Bird Attractor"
-Date "2016-01-30"
-Rev "A"
-Comp "MITTO DESIGN LLC"
-Comment1 "Matthew Swarts"
-Comment2 "Rachel LeRoy"
+Date "2016-10-24"
+Rev "C"
+Comp "Matthew Swarts and Racel LeRoy"
+Comment1 "MIT License"
+Comment2 ""
 Comment3 ""
 Comment4 ""
@@
 F 0 "SW1" H 2250 3535 50  0000 C CNN
 F 1 "SW_PUSH" H 2100 3345 50  0000 C CNN
-F 2 "Buttons_Switches_SMD:SW_SPST_PTS645" H 2100 3425 50  0001 C CNN
+F 2 "Buttons_Switches_ThroughHole:SW_PUSH_SMALL" H 2100 3425 50  0001 C CNN
 F 3 "" H 2100 3425 50  0000 C CNN
 	1    2100 3425
@@
 F 3 "" H 5325 1225 50  0000 C CNN
 	1    5325 1225
-	1    0    0    -1
-$EndComp
-$Comp
-L SN74LVC1G14 U3
-U 1 1 57FE78B8
-P 1875 5200
-F 0 "U3" H 1875 5300 60  0000 C CNN
-F 1 "SN74LVC1G14" H 1875 5150 60  0000 C CNN
-F 2 "MyKiCadParts:SOT-23-5-80" H 1875 5200 60  0001 C CNN
-F 3 "" H 1875 5200 60  0000 C CNN
-	1    1875 5200
-	1    0    0    -1
-$EndComp
-$Comp
-L PCF2129AT U5
-U 1 1 57FE8569
-P 1900 5550
-F 0 "U5" H 1900 5500 60  0000 C CNN
-F 1 "PCF2129AT" H 1850 5650 60  0000 C CNN
-F 2 "MyKiCadParts:SOIC-20_7.5x12.8mm_Pitch1.27mm-80" H 1900 5550 60  0001 C CNN
-F 3 "" H 1900 5550 60  0000 C CNN
-	1    1900 5550
 	1    0    0    -1
 $EndComp
@@
 P 3475 6100
 F 0 "R9" V 3555 6100 50  0000 C CNN
-F 1 "100K" V 3475 6100 50  0000 C CNN
+F 1 "10K" V 3475 6100 50  0000 C CNN
 F 2 "Capacitors_SMD:C_1206" V 3405 6100 50  0001 C CNN
 F 3 "" H 3475 6100 50  0000 C CNN
@@
 P 3475 1425
 F 0 "C1" H 3500 1525 50  0000 L CNN
-F 1 "1uF" H 3500 1325 50  0000 L CNN
+F 1 "10uF" H 3500 1325 50  0000 L CNN
 F 2 "Capacitors_SMD:C_0805" H 3513 1275 50  0001 C CNN
 F 3 "" H 3475 1425 50  0000 C CNN
@@
 5V_IN
 Wire Wire Line
-	6775 3100 6775 3200
-Wire Wire Line
-	6675 3150 6975 3150
-Wire Wire Line
-	6975 3150 6975 3250
-Connection ~ 6775 3150
+	6975 2750 6975 3250
 Wire Wire Line
 	6775 3500 6775 3550
@@
 Wire Wire Line
 	9725 4125 9775 4125
-Text GLabel 9775 3825 2    60   Input ~ 0
+Text GLabel 9725 3825 2    60   Input ~ 0
 GND
 $Comp
@@
 	2350 3075 2350 3125
 $Comp
-L R R20
-U 1 1 58036BD3
-P 6775 2950
-F 0 "R20" V 6855 2950 50  0000 C CNN
-F 1 "0" V 6775 2950 50  0000 C CNN
-F 2 "Resistors_SMD:R_1206" V 6705 2950 50  0001 C CNN
-F 3 "" H 6775 2950 50  0000 C CNN
-	1    6775 2950
-	1    0    0    -1
-$EndComp
-Wire Wire Line
-	6775 2700 6775 2800
-Wire Wire Line
-	6675 3150 6675 2750
-Wire Wire Line
-	6675 2750 6775 2750
-Connection ~ 6775 2750
-$Comp
 L R R21
 U 1 1 580EDD4C
@@
 Text GLabel 5400 3550 2    60   Input ~ 0
 V33
+Wire Wire Line
+	6775 3200 6775 2700
+Wire Wire Line
+	6975 2750 6775 2750
+Connection ~ 6775 2750
 $EndSCHEMATC
